File: sweet-sixteen.sch (KiCad schematic (older format))
At the start: 35 parts

Commit message: add power in, pi note and pi interface
Parts:
- added CON?: PWR, symbol BARREL_JACK
- added F?: 500mA, symbol F_Small
- added P?: RPI_IF, symbol CONN_02X40
Connections:
- net GND: now also CON?.2, P?.14 (P14), P?.25 (P25), P?.6 (P6)
- net VCC: no longer P?.1 (P1), P?.1 (P1)
- net SDA: now reaches P?.1 (P1), U?.2 (SDI)
- net SDA: now also P?.19 (P19)
- net CLK: now reaches P?.1 (P1), P?.1 (P1), U?.3 (CLK), U?.3 (CLK), U?.3 (CLK), U?.3 (CLK), U?.3 (CLK), U?.3 (CLK), U?.3 (CLK), U?.3 (CLK)
- net CLK: now also P?.23 (P23)
- net LE: now reaches P?.1 (P1), P?.1 (P1), U?.4 (LE), U?.4 (LE), U?.4 (LE), U?.4 (LE), U?.4 (LE), U?.4 (LE), U?.4 (LE), U?.4 (LE)
- net LE: now also P?.15 (P15)
- new net: F?.1, P?.2 (P2)
- new net +5V: CON?.1, F?.2, P?.1 (P1), P?.1 (P1)
Other:
- note added: "Note:\nOne the first of the multiple Display-Boards,\nthe RPi-Section is populated, while on the other\nboards it can simply be left Blank.\n\nIt contains an RPi Extension Port Socket, which\nconnects the RPis SPI-Port to the Shift-Registers\nand GPIO 22 to the LE Line of all Boards. It also\npowers the RPi from the Plugpack via the existing\nBarrel Connector.\n\nThe Local Regulator for the 3V3 R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"
Changed lines of the file:
@@
-$EndComp
-$Comp
-L VCC #PWR?
-U 1 1 584E6FF4
-P 1150 4900
-F 0 "#PWR?" H 1150 4750 50  0001 C CNN
-F 1 "VCC" H 1150 5050 50  0000 C CNN
-F 2 "" H 1150 4900 50  0000 C CNN
-F 3 "" H 1150 4900 50  0000 C CNN
-	1    1150 4900
-	1    0    0    -1
 $EndComp
 $Comp
@@
 $EndComp
 $Comp
-L VCC #PWR?
-U 1 1 584E732B
-P 15350 4900
-F 0 "#PWR?" H 15350 4750 50  0001 C CNN
-F 1 "VCC" H 15350 5050 50  0000 C CNN
-F 2 "" H 15350 4900 50  0000 C CNN
-F 3 "" H 15350 4900 50  0000 C CNN
-	1    15350 4900
-	-1   0    0    -1
-$EndComp
-$Comp
 L GND #PWR?
 U 1 1 584E7331
@@
 Wire Wire Line
 	15350 4900 15500 4900
+$Comp
+L CONN_02X40 P?
+U 1 1 584E8302
+P 2750 10200
+F 0 "P?" H 2750 12250 50  0000 C CNN
+F 1 "RPI_IF" V 2750 10200 50  0000 C CNN
+F 2 "" H 2750 10200 50  0000 C CNN
+F 3 "" H 2750 10200 50  0000 C CNN
+	1    2750 10200
+	0    1    1    0
+$EndComp
+$Comp
+L GND #PWR?
+U 1 1 584E8B98
+P 4500 10550
+F 0 "#PWR?" H 4500 10300 50  0001 C CNN
+F 1 "GND" H 4500 10400 50  0000 C CNN
+F 2 "" H 4500 10550 50  0000 C CNN
+F 3 "" H 4500 10550 50  0000 C CNN
+	1    4500 10550
+	1    0    0    -1
+$EndComp
+$Comp
+L GND #PWR?
+U 1 1 584E8F0A
+P 4100 10550
+F 0 "#PWR?" H 4100 10300 50  0001 C CNN
+F 1 "GND" H 4100 10400 50  0000 C CNN
+F 2 "" H 4100 10550 50  0000 C CNN
+F 3 "" H 4100 10550 50  0000 C CNN
+	1    4100 10550
+	1    0    0    -1
+$EndComp
+Wire Wire Line
+	4500 10550 4500 10450
+Wire Wire Line
+	4100 10550 4100 10450
+$Comp
+L +5V #PWR?
+U 1 1 584E95E2
+P 4900 10450
+F 0 "#PWR?" H 4900 10300 50  0001 C CNN
+F 1 "+5V" H 4900 10590 50  0000 C CNN
+F 2 "" H 4900 10450 50  0000 C CNN
+F 3 "" H 4900 10450 50  0000 C CNN
+	1    4900 10450
+	1    0    0    -1
+$EndComp
+Wire Wire Line
+	4900 10450 4900 10650
+Wire Wire Line
+	4700 10450 4700 10650
+Text Notes 5600 10950 0    60   ~ 0
+Note:\nOne the first of the multiple Display-Boards,\nthe RPi-Section is populated, while on the other\nboards it can simply be left Blank.\n\nIt contains an RPi Extension Port Socket, which\nconnects the RPis SPI-Port to the Shift-Registers\nand GPIO 22 to the LE Line of all Boards. It also\npowers the RPi from the Plugpack via the existing\nBarrel Connector.\n\nThe Local Regulator for the 3V3 Rail, which is used\nby the Shift-Registers as Supply and the 4V2 Rail which\npowers the LEDs must be populated on all Boards.
+$Comp
+L +5V #PWR?
+U 1 1 584EF84A
+P 15350 4900
+F 0 "#PWR?" H 15350 4750 50  0001 C CNN
+F 1 "+5V" H 15350 5040 50  0000 C CNN
+F 2 "" H 15350 4900 50  0000 C CNN
+F 3 "" H 15350 4900 50  0000 C CNN
+	1    15350 4900
+	1    0    0    -1
+$EndComp
+$Comp
+L +5V #PWR?
+U 1 1 584EF95E
+P 1150 4900
+F 0 "#PWR?" H 1150 4750 50  0001 C CNN
+F 1 "+5V" H 1150 5040 50  0000 C CNN
+F 2 "" H 1150 4900 50  0000 C CNN
+F 3 "" H 1150 4900 50  0000 C CNN
+	1    1150 4900
+	1    0    0    -1
+$EndComp
+$Comp
+L BARREL_JACK CON?
+U 1 1 584F0BF1
+P 950 5850
+F 0 "CON?" H 950 6100 50  0000 C CNN
+F 1 "PWR" H 950 5650 50  0000 C CNN
+F 2 "" H 950 5850 50  0000 C CNN
+F 3 "" H 950 5850 50  0000 C CNN
+	1    950  5850
+	1    0    0    -1
+$EndComp
+$Comp
+L GND #PWR?
+U 1 1 584F0CCF
+P 1250 6100
+F 0 "#PWR?" H 1250 5850 50  0001 C CNN
+F 1 "GND" H 1250 5950 50  0000 C CNN
+F 2 "" H 1250 6100 50  0000 C CNN
+F 3 "" H 1250 6100 50  0000 C CNN
+	1    1250 6100
+	1    0    0    -1
+$EndComp
+$Comp
+L +5V #PWR?
+U 1 1 584F0D49
+P 1250 5600
+F 0 "#PWR?" H 1250 5450 50  0001 C CNN
+F 1 "+5V" H 1250 5740 50  0000 C CNN
+F 2 "" H 1250 5600 50  0000 C CNN
+F 3 "" H 1250 5600 50  0000 C CNN
+	1    1250 5600
+	1    0    0    -1
+$EndComp
+Wire Wire Line
+	1250 5600 1250 5750
+Wire Wire Line
+	1250 5950 1250 6100
+$Comp
+L F_Small F?
+U 1 1 584F1690
+P 4800 10650
+F 0 "F?" H 4760 10710 50  0000 L CNN
+F 1 "500mA" H 4680 10590 50  0000 L CNN
+F 2 "" H 4800 10650 50  0000 C CNN
+F 3 "" H 4800 10650 50  0000 C CNN
+	1    4800 10650
+	1    0    0    -1
+$EndComp
+Wire Notes Line
+	8550 11250 8550 9200
+Wire Notes Line
+	8550 9200 450  9200
+Text Label 1550 4400 0    60   ~ 0
+CLK
+Text Label 1550 4550 0    60   ~ 0
+LE
+Text Label 1000 4050 1    60   ~ 0
+SDA
+Wire Wire Line
+	3800 9950 3800 9550
+Text Label 3800 9700 1    60   ~ 0
+SDA
+Wire Wire Line
+	3600 9950 3600 9550
+Text Label 3600 9700 1    60   ~ 0
+CLK
+$Comp
+L GND #PWR?
+U 1 1 584F504F
+P 3500 9900
+F 0 "#PWR?" H 3500 9650 50  0001 C CNN
+F 1 "GND" H 3500 9750 50  0000 C CNN
+F 2 "" H 3500 9900 50  0000 C CNN
+F 3 "" H 3500 9900 50  0000 C CNN
+	1    3500 9900
+	-1   0    0    1
+$EndComp
+Wire Wire Line
+	3500 9900 3500 9950
+Wire Wire Line
+	4000 9950 4000 9550
+Text Label 4000 9650 1    60   ~ 0
+LE
 $EndSCHEMATC

Commit message: add level shifter, power net, 9th driver
Parts:
- removed U?: STP16CPC26, symbol STP16CPC26
- added C? (x10): 10nf, symbol C_Small
- added C?: 100nf, symbol C_Small
- added D? (x8): LED, symbol LED
- added JP1: JUMPER, symbol JUMPER
- added P?: 5V_I, symbol CONN_01X01
- added P?: 5V_O, symbol CONN_01X01
- added R?: R, symbol R
- added U?: STP16CPC26, symbol STP16CPC26
- added U? (x4): 74LS08, symbol 74LS08
- added U? (x2): LM7808ACT, TO-220, symbol LM7808ACT
- added W?: +12V, symbol TEST_1P
- added W?: +5V, symbol TEST_1P
- added W?: GND, symbol TEST_1P
- added W?: VLED, symbol TEST_1P
- P?: value VCC_I -> 12V_I
- P?: value VCC_O -> 12V_O
- gave numbers to parts that had none: 1
Connections:
- net CLK: now also U?.3 (CLK), U?.3, U?.3 (CLK); no longer P?.23 (P23)
- net GND: now also U?.1 (GND), U?.21 (~OE), C?.2, C?.2, C?.2, C?.2, C?.2, C?.2, C?.2, C?.2, C?.2, C?.2, C?.2, R?.1, U?.1 (GND), U?.2 (GND), U?.2 (GND), U?.21 (~OE), U?.7 (GND), U?.7 (GND), U?.7 (GND), U?.7 (GND), W?.1
- net LE: now also U?.4 (LE), JP1.2, U?.4 (LE), U?.8; no longer P?.15 (P15)
- net SDA: now also U?.6; no longer P?.19 (P19)
- net VCC: now also F?.2, U?.24 (VDD), C?.1, C?.1, C?.1, C?.1, C?.1, C?.1, C?.1, C?.1, C?.1, C?.1, C?.1, P?.1 (P1), P?.1 (P1), U?.14 (VCC), U?.14 (VCC), U?.14 (VCC), U?.14 (VCC), U?.24 (VDD), U?.3 (OUT), W?.1
- net VLED: now reaches AFF?.11 (C.A.)
- net VLED: now also AFF?.11 (C.A.), AFF?.11 (C.A.), AFF?.11 (C.A.), AFF?.11 (C.A.), AFF?.11 (C.A.), AFF?.11 (C.A.), AFF?.11 (C.A.), D?.2 (A), D?.2 (A), D?.2 (A), D?.2 (A), D?.2 (A), D?.2 (A), D?.2 (A), D?.2 (A), U?.3 (OUT), W?.1
- net at AFF?.12 (DP): now also U?.12 (OUT7)
- net at AFF?.12 (DP): now also U?.11 (OUT6)
- net at AFF?.12 (DP): now also U?.10 (OUT5)
- net at AFF?.12 (DP): now also U?.9 (OUT4)
- net at AFF?.12 (DP): now also U?.8 (OUT3)
- net at AFF?.12 (DP): now also U?.7 (OUT2)
- net at AFF?.12 (DP): now also U?.6 (OUT1)
- net at AFF?.1 (a): now also U?.5 (OUT0)
- net at AFF?.10 (e): now also U?.9 (OUT4)
- net at AFF?.12 (DP): now also U?.5 (OUT0)
- net at AFF?.13 (d): now also U?.8 (OUT3)
- net at AFF?.14 (r): now also U?.18 (OUT13)
- net at AFF?.15 (p): now also U?.16 (OUT11)
- net at AFF?.16 (c): now also U?.7 (OUT2)
- net at AFF?.17 (n): now also U?.15 (OUT10)
- net at AFF?.18 (b): now also U?.6 (OUT1)
- net at AFF?.2 (m): now also U?.14 (OUT9)
- net at AFF?.3 (k): now also U?.13 (OUT8)
- net at AFF?.4 (h): now also U?.12 (OUT7)
- net at AFF?.5 (u): now also U?.20 (OUT15)
- net at AFF?.6 (s): now also U?.17 (OUT12)
- net at AFF?.7 (t): now also U?.19 (OUT14)
- net at AFF?.8 (g): now also U?.11 (OUT6)
- net at AFF?.9 (f): now also U?.10 (OUT5)
- net at U?.22 (SDO): now also U?.2 (SDI)
- net at P?.1 (P1): now also U?.22 (SDO), JP1.1
- net at R?.2: now also U?.23 (R-EXT)
- net at U?.13 (OUT8): now also D?.1 (K)
- net at U?.14 (OUT9): now also D?.1 (K)
- net at U?.15 (OUT10): now also D?.1 (K)
- net at U?.16 (OUT11): now also D?.1 (K)
- net at U?.17 (OUT12): now also D?.1 (K)
- net at U?.18 (OUT13): now also D?.1 (K)
- net at U?.19 (OUT14): now also D?.1 (K)
- net at U?.2 (SDI): now also U?.22 (SDO)
- net at U?.20 (OUT15): now also D?.1 (K)
- net at U?.23 (R-EXT): now also R?.2
- net +5V renamed +12V
- net +12V: now also U?.1 (IN), U?.1 (IN), W?.1; no longer F?.2, P?.1 (P1)
- new net: P?.15 (P15), U?.10, U?.9
- new net: P?.19 (P19), U?.4, U?.5
- new net: P?.23 (P23), U?.1, U?.2
- new net: U?.12, U?.13
- no-connect marks 0 -> 1
Other:
- note added: "Note: 7805 are only examples here,\nneed to be replaced with proper\nDC-DC converters, once the required\nvoltages and aperages are known"
- note added: "Note: 8A Campable Trace between\n12V_I, 12VO resp. GND_I, GND_O\nand CON_PWR"
- note added: "Note: 8th Driver for Decimal Points\nand Aux-LEDs might not be populated.\nThen, JP1 must be bridged to connedt\nSDA to SDO directly"
- note added: "Note:\nOne the first of the multiple Display-Boards,\nthe RPi-Section is populated, while on the other\nboards it can simply be left Blank.\n\nIt contains an RPi Extension Port Socket, which\nconnects the RPis SPI-Port via a Level-Shifter to\nthe Shift-Registers and GPIO 22 to the LE Line of\nall Boards. It also powers the RPi from the 5V for\nthe Shift-Registers, which is generated from the#\n12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"
- note added: "POWER"
- note added: "RPi Interface"
- note removed: "Note:\nOne the first of the multiple Display-Boards,\nthe RPi-Section is populated, while on the other\nboards it can simply be left Blank.\n\nIt contains an RPi Extension Port Socket, which\nconnects the RPis SPI-Port to the Shift-Registers\nand GPIO 22 to the LE Line of all Boards. It also\npowers the RPi from the Plugpack via the existing\nBarrel Connector.\n\nThe Local Regulator for the 3V3 R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"
- moved on the sheet: AFF?, CON_PWR, F?, P?, R?, U?

Commit message: make more use of unused space
Other:
- note added: "Voltage Testpoints"
- moved on the sheet: CON_PWR, P?, U?, U?A, U?B, U?C, U?D, W?

Commit message: make even more use out of that unused space
Connections:
- net LE: no longer JP1.2
- net at U?.2 (SDI), U?.22 (SDO): now also JP1.2
Other:
- moved on the sheet: C?, D?, JP1, R?, U?
